File: ethercon_breakout.kicad_sch (KiCad schematic)
At the start: 5 parts, among them J101 NE8FAH, J102 ORANGE, J103 GREEN, J104 BLUE, J105 BROWN

Commit message: Changed schematic title
Other:
- company: (none) -> Marek Jansky
- title: (none) -> Ethercon breakout board
Changed lines of the file:
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@@
 (kicad_sch (version 20230121) (generator eeschema)
   (paper "A4")
+  (title_block
+    (title "Ethercon breakout board")
+    (date "2024-03-12")
+    (rev "1")
+    (company "Marek Jansky")
+  )
   (junction (at 114.3 76.2) (diameter 0) (color 0 0 0 0)
   )
